Commit message: Change tags position - update x y and z/

File: urdf/tag_13.urdf.xacro (robot description, xacro)
@@ -1,10 +1,26 @@
 <?xml version="1.0"?>
-<robot name="tags_13" xmlns:xacro="http://ros.org/wiki/xacro">
+<robot name="tag_13_settings" xmlns:xacro="http://ros.org/wiki/xacro">
+<!-- Measured distances between tags -->
+<xacro:property name="dx" value="1.53" />
+<xacro:property name="dy" value="0" />
+<xacro:property name="dz" value="0.05" />
+  <!-- Below goes the description of either a link that is close to the tag_13, which will be named "near_13"
+  or the description of a link that is close to another tag, which will be used to send the robot elsewhere -->
+  <!-- The link which the will be seen by the marker localizator -->
   <link name="tag_13"/>
+  <!-- A link for a 'near tag' pose setting purpose: -->
   <link name="near_13"/>
   <joint name="tag13_joint_to_near_13" type="fixed">
     <origin xyz="0 0 0.3" rpy="0 0 0"/>
-    <parent link="tag_13"/>
+    <parent link="tag_13"/>tags_13
     <child link="near_13"/>
   </joint>
+  <!-- A link to send the robot close to another tag -->
+  <link name="goal_tag_14"/>
+  <joint name="forward_to_tag_14" type="fixed">
+  <!-- The origin must have the coordinates to a point near tag 14. This must be measured and entered beforehand -->
+    <origin xyz="${dx} ${dy} ${dz}" rpy="0 0 0"/>
+    <parent link="tag_13"/>
+    <child link="goal_tag_14"/>
+  </joint>
 </robot>

File: urdf/tag_14.urdf.xacro (robot description, xacro)
@@ -1,5 +1,12 @@
 <?xml version="1.0"?>
-<robot name="tags_14" xmlns:xacro="http://ros.org/wiki/xacro">
+<robot name="tag_14_settings" xmlns:xacro="http://ros.org/wiki/xacro">
+<xacro:property name="dx" value="2.25" />
+<xacro:property name="dy" value="0" />
+<xacro:property name="dz" value="1.35" />
+  <!-- Below goes the description of either a link that is close to the tag_14, which will be named "near_13"
+  or the description of a link that is close to another tag, which will be used to send the robot elsewhere -->
+  <!-- The link which the will be seen by the marker localizator -->
   <link name="tag_14"/>
+  <!-- A link for a 'near tag' pose setting purpose: -->
   <link name="near_14"/>
   <joint name="tag14_joint_to_near_14" type="fixed">
@@ -8,3 +15,11 @@
     <child link="near_14"/>
   </joint>
+  <!-- A link to send the robot close to another tag -->
+  <link name="goal_tag_15"/>
+  <joint name="forward_to_tag_15" type="fixed">
+  <!-- The origin must have the coordinates to a point near tag 14. This must be measured and entered beforehand -->
+    <origin xyz="${dx} ${dy} ${dz}" rpy="0 0 0"/>
+    <parent link="tag_14"/>
+    <child link="goal_tag_15"/>
+  </joint>
 </robot>

File: urdf/tag_15.urdf.xacro (robot description, xacro)
@@ -1,10 +1,25 @@
 <?xml version="1.0"?>
-<robot name="tags_15" xmlns:xacro="http://ros.org/wiki/xacro">
+<robot name="tag_15_settings" xmlns:xacro="http://ros.org/wiki/xacro">
+<xacro:property name="dx" value="-1.3" />
+<xacro:property name="dy" value="0.0" />
+<xacro:property name="dz" value="3.8" />
+  <!-- Below goes the description of either a link that is close to the tag_13, which will be named "near_13"
+  or the description of a link that is close to another tag, which will be used to send the robot elsewhere -->
+  <!-- The link which the will be seen by the marker localizator -->
   <link name="tag_15"/>
+  <!-- A link for a 'near tag' pose setting purpose: -->
   <link name="near_15"/>
-  <joint name="tag15_joint_to_near_15" type="fixed">
+  <joint name="tag13_joint_to_near_13" type="fixed">
     <origin xyz="0 0 0.3" rpy="0 0 0"/>
     <parent link="tag_15"/>
     <child link="near_15"/>
   </joint>
+  <!-- A link to send the robot close to another tag -->
+  <link name="goal_tag_13"/>
+  <joint name="forward_to_tag_13" type="fixed">
+  <!-- The origin must have the coordinates to a point near tag 14. This must be measured and entered beforehand -->
+    <origin xyz="${dx} ${dy} ${dz}" rpy="0 0 0"/>
+    <parent link="tag_15"/>
+    <child link="goal_tag_13"/>
+  </joint>
 </robot>

Commit message: Change the 'near_tag' distance to 30 cm

File: urdf/tag_13.urdf.xacro (robot description, xacro)
@@ -4,5 +4,5 @@
 <xacro:property name="dx" value="1.53" />
 <xacro:property name="dy" value="0" />
-<xacro:property name="dz" value="0.05" />
+<xacro:property name="dz" value="0.20" />
   <!-- Below goes the description of either a link that is close to the tag_13, which will be named "near_13"
   or the description of a link that is close to another tag, which will be used to send the robot elsewhere -->
@@ -13,5 +13,5 @@
   <joint name="tag13_joint_to_near_13" type="fixed">
     <origin xyz="0 0 0.3" rpy="0 0 0"/>
-    <parent link="tag_13"/>tags_13
+    <parent link="tag_13"/>
     <child link="near_13"/>
   </joint>
@@ -21,5 +21,5 @@
   <!-- The origin must have the coordinates to a point near tag 14. This must be measured and entered beforehand -->
     <origin xyz="${dx} ${dy} ${dz}" rpy="0 0 0"/>
-    <parent link="tag_13"/>
+    <parent link="near_13"/>
     <child link="goal_tag_14"/>
   </joint>

File: urdf/tag_14.urdf.xacro (robot description, xacro)
@@ -1,7 +1,7 @@
 <?xml version="1.0"?>
 <robot name="tag_14_settings" xmlns:xacro="http://ros.org/wiki/xacro">
-<xacro:property name="dx" value="2.25" />
+<xacro:property name="dx" value="1.8" />
 <xacro:property name="dy" value="0" />
-<xacro:property name="dz" value="1.35" />
+<xacro:property name="dz" value="0.9" />
   <!-- Below goes the description of either a link that is close to the tag_14, which will be named "near_13"
   or the description of a link that is close to another tag, which will be used to send the robot elsewhere -->
@@ -20,5 +20,5 @@
   <!-- The origin must have the coordinates to a point near tag 14. This must be measured and entered beforehand -->
     <origin xyz="${dx} ${dy} ${dz}" rpy="0 0 0"/>
-    <parent link="tag_14"/>
+    <parent link="near_14"/>
     <child link="goal_tag_15"/>
   </joint>

File: urdf/tag_15.urdf.xacro (robot description, xacro)
@@ -1,5 +1,5 @@
 <?xml version="1.0"?>
 <robot name="tag_15_settings" xmlns:xacro="http://ros.org/wiki/xacro">
-<xacro:property name="dx" value="-1.3" />
+<xacro:property name="dx" value="-1.0" />
 <xacro:property name="dy" value="0.0" />
 <xacro:property name="dz" value="3.8" />
@@ -20,5 +20,5 @@
   <!-- The origin must have the coordinates to a point near tag 14. This must be measured and entered beforehand -->
     <origin xyz="${dx} ${dy} ${dz}" rpy="0 0 0"/>
-    <parent link="tag_15"/>
+    <parent link="near_15"/>
     <child link="goal_tag_13"/>
   </joint>
